File: stacja_pomiarowa/schemat/stacja_pomiarowa_panel/czujniki_dht11_ds18b20.kicad_sch (KiCad schematic)
At the start: 16 parts, among them J20 Conn_01x03, J21 Conn_01x03, J22 Conn_01x03, J23 Conn_01x03, J24 Conn_01x03

Commit message: Dodano ledy informujące czy urządzenie połączyło się z systemem, dodane tytuły podschematów ze złączami
Other:
- title: (none) -> Złącza dla czujników cyfrowych
Changed lines of the file:
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@@
 (kicad_sch (version 20230121) (generator eeschema)
   (paper "A5")
+  (title_block
+    (title "Złącza dla czujników cyfrowych")
+  )
   (junction (at 125.095 39.37) (diameter 0) (color 0 0 0 0)
   )
