File: stacja_pomiarowa/schemat/stacja_pomiarowa_panel/stacja_pomiarowa_panel.kicad_sch (KiCad schematic)
At the start: 5 parts, among them J17 Conn_02x08_Counter_Clockwise, J18 Conn_01x04, J19 Conn_02x17_Counter_Clockwise, J52 Conn_02x04_Counter_Clockwise, J61 Conn_01x01

Commit message: Zmiana złącza zasilania do panela z 4-pinowego na 2-pinowe
Parts:
- removed J18: Conn_01x04, symbol Connector_Generic:Conn_01x04
- added J18: Conn_01x02, symbol Connector_Generic:Conn_01x02
Connections:
- net +5V: now also J18.1 (Pin_1)
- net GND: now also J18.2 (Pin_2)
Changed lines of the file:
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@@
 (kicad_sch (version 20230121) (generator eeschema)
   (paper "A5")
-  (junction (at 16.51 120.015) (diameter 0) (color 0 0 0 0)
-  )
-  (junction (at 21.59 125.095) (diameter 0) (color 0 0 0 0)
-  )
   (no_connect (at 160.655 57.785))
   (no_connect (at 160.655 60.325))
@@
     (stroke (width 0) (type default))
   )
-  (wire (pts (xy 24.765 125.095) (xy 21.59 125.095))
-    (stroke (width 0) (type default))
-  )
   (wire (pts (xy 29.845 97.79) (xy 60.96 97.79))
     (stroke (width 0) (type default))
@@
     (stroke (width 0) (type default))
   )
-  (wire (pts (xy 16.51 119.38) (xy 16.51 120.015))
-    (stroke (width 0) (type default))
-  )
-  (wire (pts (xy 24.765 122.555) (xy 16.51 122.555))
-    (stroke (width 0) (type default))
-  )
-  (wire (pts (xy 16.51 120.015) (xy 24.765 120.015))
-    (stroke (width 0) (type default))
-  )
   (wire (pts (xy 71.12 22.86) (xy 67.945 22.86))
     (stroke (width 0) (type default))
@@
     (stroke (width 0) (type default))
   )
-  (wire (pts (xy 24.765 117.475) (xy 21.59 117.475))
-    (stroke (width 0) (type default))
-  )
   (wire (pts (xy 170.18 42.545) (xy 160.655 42.545))
     (stroke (width 0) (type default))
@@
     (stroke (width 0) (type default))
   )
-  (wire (pts (xy 16.51 120.015) (xy 16.51 122.555))
-    (stroke (width 0) (type default))
-  )
   (wire (pts (xy 29.845 85.09) (xy 57.785 85.09))
     (stroke (width 0) (type default))
   )
-  (wire (pts (xy 21.59 117.475) (xy 21.59 125.095))
-    (stroke (width 0) (type default))
-  )
   (wire (pts (xy 59.055 69.85) (xy 53.975 69.85))
     (stroke (width 0) (type default))
@@
     (stroke (width 0) (type default))
   )
-  (wire (pts (xy 21.59 125.095) (xy 21.59 125.73))
-    (stroke (width 0) (type default))
-  )
   (wire (pts (xy 133.985 40.005) (xy 147.955 40.005))
     (stroke (width 0) (type default))
@@
     (stroke (width 0) (type default))
   )
-  (symbol (lib_id "Connector_Generic:Conn_01x04") (at 29.845 120.015 0) (unit 1)
-    (in_bom yes) (on_board yes) (dnp no) (fields_autoplaced)
-    (property "Reference" "J18" (at 33.02 120.65 0)
-      (effects (font (size 1.27 1.27)) (justify left))
-    )
-    (property "Value" "Conn_01x04" (at 33.02 123.19 0)
-      (effects (font (size 1.27 1.27)) (justify left))
-    )
-    (property "Footprint" "" (at 29.845 120.015 0)
-      (effects (font (size 1.27 1.27)) hide)
-    )
-    (property "Datasheet" "~" (at 29.845 120.015 0)
-      (effects (font (size 1.27 1.27)) hide)
-    )
-    (pin "1")
-    (pin "2")
-    (pin "3")
-    (pin "4")
-    (instances
-      (project "stacja_pomiarowa_panel"
-        (path "/b68efdb9-d9e6-4201-adfc-9623b369d78a"
-          (reference "J18") (unit 1)
-        )
-      )
-    )
-  )
   (symbol (lib_id "power:+5V") (at 58.42 121.285 0) (unit 1)
     (in_bom yes) (on_board yes) (dnp no) (fields_autoplaced)
@@
     )
   )
-  (symbol (lib_id "power:+5V") (at 16.51 119.38 0) (unit 1)
-    (in_bom yes) (on_board yes) (dnp no) (fields_autoplaced)
-    (property "Reference" "#PWR033" (at 16.51 123.19 0)
-      (effects (font (size 1.27 1.27)) hide)
-    )
-    (property "Value" "+5V" (at 16.51 115.57 0)
-      (effects (font (size 1.27 1.27)))
-    )
-    (property "Footprint" "" (at 16.51 119.38 0)
-      (effects (font (size 1.27 1.27)) hide)
-    )
-    (property "Datasheet" "" (at 16.51 119.38 0)
+  (symbol (lib_id "power:+5V") (at 25.654 122.428 0) (unit 1)
+    (in_bom yes) (on_board yes) (dnp no) (fields_autoplaced)
+    (property "Reference" "#PWR033" (at 25.654 126.238 0)
+      (effects (font (size 1.27 1.27)) hide)
+    )
+    (property "Value" "+5V" (at 25.654 118.618 0)
+      (effects (font (size 1.27 1.27)))
+    )
+    (property "Footprint" "" (at 25.654 122.428 0)
+      (effects (font (size 1.27 1.27)) hide)
+    )
+    (property "Datasheet" "" (at 25.654 122.428 0)
       (effects (font (size 1.27 1.27)) hide)
     )
@@
         (path "/b68efdb9-d9e6-4201-adfc-9623b369d78a"
           (reference "J61") (unit 1)
+        )
+      )
+    )
+  )
+  (symbol (lib_id "Connector_Generic:Conn_01x02") (at 30.734 122.428 0) (unit 1)
+    (in_bom yes) (on_board yes) (dnp no) (fields_autoplaced)
+    (property "Reference" "J18" (at 33.02 123.063 0)
+      (effects (font (size 1.27 1.27)) (justify left))
+    )
+    (property "Value" "Conn_01x02" (at 33.02 125.603 0)
+      (effects (font (size 1.27 1.27)) (justify left))
+    )
+    (property "Footprint" "" (at 30.734 122.428 0)
+      (effects (font (size 1.27 1.27)) hide)
+    )
+    (property "Datasheet" "~" (at 30.734 122.428 0)
+      (effects (font (size 1.27 1.27)) hide)
+    )
+    (pin "1")
+    (pin "2")
+    (instances
+      (project "stacja_pomiarowa_panel"
+        (path "/b68efdb9-d9e6-4201-adfc-9623b369d78a"
+          (reference "J18") (unit 1)
         )
       )
@@
     )
   )
-  (symbol (lib_id "power:GND") (at 21.59 125.73 0) (unit 1)
-    (in_bom yes) (on_board yes) (dnp no) (fields_autoplaced)
-    (property "Reference" "#PWR034" (at 21.59 132.08 0)
-      (effects (font (size 1.27 1.27)) hide)
-    )
-    (property "Value" "GND" (at 21.59 130.81 0)
-      (effects (font (size 1.27 1.27)))
-    )
-    (property "Footprint" "" (at 21.59 125.73 0)
-      (effects (font (size 1.27 1.27)) hide)
-    )
-    (property "Datasheet" "" (at 21.59 125.73 0)
-      (effects (font (size 1.27 1.27)) hide)
-    )
+  (symbol (lib_id "power:GND") (at 25.654 124.968 0) (unit 1)
+    (in_bom yes) (on_board yes) (dnp no) (fields_autoplaced)
+    (property "Reference" "#PWR034" (at 25.654 131.318 0)
+      (effects (font (size 1.27 1.27)) hide)
+    )
+    (property "Value" "GND" (at 25.654 130.048 0)
+      (effects (font (size 1.27 1.27)))
+    )
+    (property "Footprint" "" (at 25.654 124.968 0)
+      (effects (font (size 1.27 1.27)) hide)
+    )
+    (property "Datasheet" "" (at 25.654 124.968 0)
+      (effects (font (size 1.27 1.27)) hide)
+    )

Commit message: Dodano ledy informujące czy urządzenie połączyło się z systemem, dodane tytuły podschematów ze złączami
Other:
- title: (none) -> Stacja pomiarowa, panel ze złączami
Changed lines of the file:
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@@
 (kicad_sch (version 20230121) (generator eeschema)
   (paper "A5")
+  (title_block
+    (title "Stacja pomiarowa, panel ze złączami")
+  )
   (no_connect (at 160.655 57.785))
   (no_connect (at 160.655 60.325))
